Commit message: Added Gazebo UR5e simulation with ros2_control

File: src/arm_sim/urdf/ur5e.urdf (robot description, URDF)
Before this commit: robot ur5e, 13 links, 12 joints
Links:
- link base_link_inertia: geometry collision mesh filename=file:///opt/ros/jazzy/share/ur_description/meshes/ur5e/coll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; visual mesh filename=file:///opt/ros/jazzy/share/ur_description/meshes/ur5e/visu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
- link forearm_link: geometry collision mesh filename=file:///opt/ros/jazzy/share/ur_description/meshes/ur5e/coll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; visual mesh filename=file:///opt/ros/jazzy/share/ur_description/meshes/ur5e/visu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
- link shoulder_link: geometry collision mesh filename=file:///opt/ros/jazzy/share/ur_description/meshes/ur5e/coll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; visual mesh filename=file:///opt/ros/jazzy/share/ur_description/meshes/ur5e/visu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
- link upper_arm_link: geometry collision mesh filename=file:///opt/ros/jazzy/share/ur_description/meshes/ur5e/coll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; visual mesh filename=file:///opt/ros/jazzy/share/ur_description/meshes/ur5e/visu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
- link wrist_1_link: geometry collision mesh filename=file:///opt/ros/jazzy/share/ur_description/meshes/ur5e/coll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; visual mesh filename=file:///opt/ros/jazzy/share/ur_description/meshes/ur5e/visu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
- link wrist_2_link: geometry collision mesh filename=file:///opt/ros/jazzy/share/ur_description/meshes/ur5e/coll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; visual mesh filename=file:///opt/ros/jazzy/share/ur_description/meshes/ur5e/visu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
- link wrist_3_link: geometry collision mesh filename=file:///opt/ros/jazzy/share/ur_description/meshes/ur5e/coll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; visual mesh filename=file:///opt/ros/jazzy/share/ur_description/meshes/ur5e/visu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
